File: pcb/HDC100X-Breakout_v10.sch (EAGLE design)
At the start: 14 parts, among them IC1 HDC100x, J1 MA05-1, X1 PASSER-07, X2 PASSER-07

Commit message: updated license infos
Other:
- note added: "Designed by Stephan Watterott (Watterott electronic)"
- note added: "Released under the Creative Commons Attribution Share-Alike License"
- note added: "http://creativecommons.org/licenses/by-sa/4.0/"
- moved on the sheet: ADR0, ADR1, C1, DRDY, IC1, J1, R1, R2, R3, R4, R5
